Commit message: fixed odom to base_link transform

File: carmajava/launch/urdf/saxton_cav_green_srx.urdf (robot description, URDF)
Before this commit: robot saxton_cav_srx, 5 links, 4 joints
Links:
- removed link pinpoint
- added link position_sensor
Joints:
- removed joint host_vehicle_to_pinpoint
- added joint host_vehicle_to_position_sensor: type fixed, parent host_vehicle, child position_sensor, origin xyz=-.5 0 -1 rpy=3.145159 0 0

Commit message: fix frame naming

File: carmajava/launch/urdf/saxton_cav_green_srx.urdf (robot description, URDF)
Before this commit: robot saxton_cav_srx, 5 links, 4 joints
Links:
- removed link position_sensor
- added link pinpoint

Commit message: adding another fix for frame name in urdf file

File: carmajava/launch/urdf/saxton_cav_green_srx.urdf (robot description, URDF)
Before this commit: robot saxton_cav_srx, 5 links, 4 joints
Joints:
- joint host_vehicle_to_position_sensor: child position_sensor -> pinpoint

Commit message: fix pinpoint urdf

File: carmajava/launch/urdf/saxton_cav_green_srx.urdf (robot description, URDF)
Before this commit: robot saxton_cav_srx, 5 links, 4 joints
Joints:
- joint host_vehicle_to_position_sensor: origin xyz=-.5 0 -1 rpy=3.145159 0 0 -> xyz=0 0 0 rpy=0 0 0

Commit message: corrected transforms

File: carmajava/launch/urdf/saxton_cav_green_srx.urdf (robot description, URDF)
Before this commit: robot saxton_cav_srx, 5 links, 4 joints
Links:
- removed link radar
- added link f_lrr_frame
- added link lf_srr_frame
- added link r_srr_frame
- added link rf_srr_frame
- added link vision_frame
Joints:
- removed joint host_vehicle_to_position_sensor
- removed joint host_vehicle_to_radar
- added joint base_link_pinpoint: type fixed, parent base_link, child pinpoint, origin xyz=0 0 0 rpy=3.145159 0 0
- added joint rear_link_f_lrr_frame: type fixed, parent base_link, child f_lrr_frame, origin xyz=3.7 0 0.43 rpy=0 0 0
- added joint rear_link_lf_srr_frame: type fixed, parent base_link, child lf_srr_frame, origin xyz=3.73 0.39 0.2 rpy=0 0 0.09
- added joint rear_link_r_srr_frame: type fixed, parent base_link, child r_srr_frame, origin xyz=-0.95 0.19 0.31 rpy=0 0 3.1
- added joint rear_link_rf_srr_frame: type fixed, parent base_link, child rf_srr_frame, origin xyz=3.73 -0.39 0.2 rpy=0 0 -0.09
- added joint rear_link_vision_frame: type fixed, parent base_link, child vision_frame, origin xyz=1.94 -0.1 1.07 rpy=0 0 0
- joint base_link_to_host_vehicle: origin xyz=0 0 0 rpy=0 0 0 -> xyz=1.524 0 -0.3556 rpy=3.145159 0 0
- joint host_vehicle_to_vehicle_front: origin xyz=1 0 -.5 rpy=3.145159 0 0 -> xyz=2.4384 0 0 rpy=3.145159 0 0

Commit message: fix urdf file for 180 degree rotation

File: carmajava/launch/urdf/saxton_cav_green_srx.urdf (robot description, URDF)
Before this commit: robot saxton_cav_srx, 9 links, 8 joints
Joints:
- joint base_link_pinpoint: origin xyz=0 0 0 rpy=3.145159 0 0 -> xyz=0 0 0 rpy=3.14159265359 0 0
- joint base_link_to_host_vehicle: origin xyz=1.524 0 -0.3556 rpy=3.145159 0 0 -> xyz=1.524 0 -0.3556 rpy=3.14159265359 0 0
- joint host_vehicle_to_vehicle_front: origin xyz=2.4384 0 0 rpy=3.145159 0 0 -> xyz=2.4384 0 0 rpy=3.14159265359 0 0

Commit message: adding bounding boxes for objects and car

File: carmajava/launch/urdf/saxton_cav_green_srx.urdf (robot description, URDF)
Before this commit: robot saxton_cav_srx, 9 links, 8 joints
Links:
- added link aabb_center; visual box size=4.88 1.5 2.2
Joints:
- added joint host_vehicle_to_aabb_center: type fixed, parent host_vehicle, child aabb_center, origin xyz=0 0 -1.1 rpy=3.14159265359 0 0
