Commit message: Update default urdf to be lexus config and fix frame bug

File: carmajava/launch/urdf/carma.urdf (robot description, URDF)
Before this commit: robot carma_srx, 10 links, 9 joints
Links:
- removed link aabb_center
- removed link f_lrr_frame
- removed link lf_srr_frame
- removed link pinpoint
- removed link r_srr_frame
- removed link rf_srr_frame
- removed link vision_frame
- added link mobileye
- added link radar_fc
- added link radar_fl
- added link radar_fr
- added link radar_rl
- added link radar_rr
- added link velodyne
Joints:
- removed joint base_link_pinpoint
- removed joint host_vehicle_to_aabb_center
- removed joint host_vehicle_to_vehicle_front
- removed joint rear_link_f_lrr_frame
- removed joint rear_link_lf_srr_frame
- removed joint rear_link_r_srr_frame
- removed joint rear_link_rf_srr_frame
- removed joint rear_link_vision_frame
- added joint base_link_to_vehicle_front: type fixed, parent base_link, child vehicle_front, origin xyz=4 0 0.57 rpy=0 0 0
- added joint lidar: type fixed, parent base_link, child velodyne, origin xyz=1.02 0 2.23 rpy=0 0 0
- added joint mobileye: type fixed, parent base_link, child mobileye, origin xyz=2.195 0 1.78 rpy=0 0 0
- added joint radar_fc: type fixed, parent base_link, child radar_fc, origin xyz=4 0 0.57 rpy=0 0 0
- added joint radar_fl: type fixed, parent base_link, child radar_fl, origin xyz=3.42 1.02 0.535 rpy=0 0 0.953
- added joint radar_fr: type fixed, parent base_link, child radar_fr, origin xyz=3.42 -1.02 0.535 rpy=0 0 -0.903
- added joint radar_rl: type fixed, parent base_link, child radar_rl, origin xyz=-0.85 1.05 0.535 rpy=0 0 2.042
- added joint radar_rr: type fixed, parent base_link, child radar_rr, origin xyz=-0.85 -1.05 0.535 rpy=0 0 -1.992
- joint base_link_to_host_vehicle: origin xyz=1.524 0 -0.3556 rpy=3.14159265359 0 0 -> xyz=3.37 0 -0.3556 rpy=3.14159265359 0 0

File: configurations/lexus_rx_450h_2019/carma.urdf (robot description, URDF)
Before this commit: robot vehicle_platform, 9 links, 9 joints
Links:
- added link vehicle_front

Commit message: Add GNSS initialization to NDT

File: carmajava/launch/urdf/carma.urdf (robot description, URDF)
Before this commit: robot vehicle_platform, 10 links, 9 joints
Links:
- added link ned_heading
- added link novatel_gnss
- added link novatel_imu
Joints:
- added joint base_link_to_novatel: type fixed, parent base_link, child novatel_gnss, origin xyz=0 0 0 rpy=0 0 0
- added joint base_link_to_novatel_imu: type fixed, parent base_link, child novatel_imu, origin xyz=0 0 0 rpy=0 0 0
- added joint gnss_to_ned_heading: type fixed, parent novatel_gnss, child ned_heading, origin xyz=0 0 0 rpy=3.14159265358979323846 0 0
