Commit message: Updates to support truck configuration

File: carmajava/launch/truck_config/saxton_cav_green_srx.urdf (robot description, URDF)
Before this commit: robot saxton_cav_srx, 10 links, 9 joints
Links:
- removed link lf_srr_frame
- removed link r_srr_frame
- removed link rf_srr_frame
- removed link vision_frame
- link aabb_center: geometry visual box size=8.74 1.5 2.362
Joints:
- removed joint rear_link_lf_srr_frame
- removed joint rear_link_r_srr_frame
- removed joint rear_link_rf_srr_frame
- removed joint rear_link_vision_frame
- joint base_link_to_host_vehicle: origin xyz=1.524 0 -0.3556 rpy=3.14159265359 0 0 -> xyz=3.37 0 -0.3556 rpy=3.14159265359 0 0
- joint host_vehicle_to_vehicle_front: origin xyz=2.4384 0 0 rpy=3.14159265359 0 0 -> xyz=4.37 0 0 rpy=3.14159265359 0 0
- joint rear_link_f_lrr_frame: origin xyz=3.7 0 0.43 rpy=0 0 0 -> xyz=7.747 0 0 rpy=0 0 0
