Commit message: Demo changes

File: carmajava/launch/cadillac_config/saxton_cav.urdf (robot description, URDF)
Before this commit: robot saxton_cav_srx, 10 links, 9 joints
Joints:
- joint host_vehicle_to_vehicle_front: origin xyz=2.4384 0 0 rpy=3.14159265359 0 0 -> xyz=3.0 0 0 rpy=3.14159265359 0 0
